Commit message: Add foot rest collision shapes

File: magni_description/urdf/magni.urdf.xacro (robot description, xacro)
@@ -171,4 +171,10 @@
   <xacro:macro name="caster_wheel" params="prefix reflect">
     <link name="${prefix}_caster_wheel">
+<!--      <visual>
+        <origin xyz="${-wheel_xpos-0.19} ${reflect*0.169} ${-wheel_r+0.04}" rpy="0 0 0" />
+        <geometry>
+          <mesh filename="package://magni_description/meshes/front_wheel.dae" />
+        </geometry>
+      </visual>    -->
       <collision>
         <origin xyz="${-wheel_xpos-0.19} ${reflect*0.169} ${-wheel_r+0.04}" rpy="0 0 0" />
@@ -185,4 +191,33 @@
   <xacro:caster_wheel prefix="left" reflect="1"/>
   <xacro:caster_wheel prefix="right" reflect="-1"/>
+  <xacro:macro name="foot_rest" params="prefix wheel_distance">
+    <link name="${prefix}_big_caster_wheel">
+      <visual>
+        <origin xyz="0 0 0" rpy="0 0 0" />
+        <geometry>
+          <mesh filename="package://magni_description/meshes/front_wheel.dae" />
+        </geometry>
+      </visual>
+      <collision>
+        <origin xyz="${3*wheel_r/4} 0 0" rpy="0 0 0" />
+        <geometry>
+          <sphere radius="${wheel_r}"/>
+        </geometry>
+      </collision>
+      <collision>
+        <origin xyz="0.07 ${-(wheel_distance+0.40)/2} ${wheel_r+.35}" rpy="0 0 0" />
+        <geometry>
+          <box size=" 0.51 ${wheel_distance+0.40} 0.70"/>
+        </geometry>
+      </collision>
+    </link>
+    <joint name="${prefix}_big_caster_wheel_joint" type="fixed">
+      <parent link="base_link"/>
+      <child link="${prefix}_big_caster_wheel"/>
+      <origin xyz="${-wheel_distance-0.31} -0.071 0" rpy="0 0 ${pi/2}"/>
+    </joint>
+  </xacro:macro>
+  <xacro:foot_rest prefix="forward" wheel_distance="0.5725"/> <!-- non-extended -->
+<!--  <xacro:foot_rest prefix="forward" wheel_distance="0.8725"/> --> <!-- extended -->
   <!-- Define all sonars, if sonars_installed set to 1 -->
   <xacro:if value="${sonars_installed}">

Commit message: Add useful reference tf links for attachment points and outer dimensions

File: magni_description/urdf/magni.urdf.xacro (robot description, xacro)
@@ -13,4 +13,5 @@
   <xacro:property name="wheel_r" value="0.1" />
   <xacro:property name="wheel_xpos" value="0.11" />
+  <xacro:property name="frame_width" value="0.2163" />
   <xacro:include filename="$(find magni_description)/urdf/magni.transmission.xacro" />
   <xacro:include filename="$(find magni_description)/urdf/magni.gazebo.xacro" />
@@ -254,3 +255,55 @@
     </xacro:ur50_lidar>
   </xacro:if>
+  <!-- Macro for robot frame points -->
+  <xacro:macro name="frame_point" params="prefix parent *origin">
+    <link name="${prefix}_point">
+<!--      <visual>
+        <origin xyz="0 0 0" rpy="0 0 0" />
+        <geometry>
+	  <sphere radius="0.01" />
+        </geometry>
+      </visual> -->
+    </link>
+    <joint name="${prefix}_point" type="fixed">
+      <parent link="${parent}"/>
+      <child link="${prefix}_point"/>
+      <xacro:insert_block name="origin"/>
+    </joint>
+  </xacro:macro>
+  <xacro:frame_point prefix="front_bottom_left" parent="base_link">
+    <origin xyz="0.089 ${-frame_width / 2} ${-wheel_r + 0.071}" rpy="0 0 0"/>
+  </xacro:frame_point>
+  <xacro:frame_point prefix="front_bottom_right" parent="base_link">
+    <origin xyz="0.089 ${frame_width / 2} ${-wheel_r + 0.071}" rpy="0 0 0"/>
+  </xacro:frame_point>
+  <xacro:frame_point prefix="back_bottom_left" parent="front_bottom_left_point">
+    <origin xyz="-0.399 0 0" rpy="0 0 0"/>
+  </xacro:frame_point>
+  <xacro:frame_point prefix="back_bottom_right" parent="front_bottom_right_point">
+    <origin xyz="-0.399 0 0" rpy="0 0 0"/>
+  </xacro:frame_point>
+  <xacro:frame_point prefix="back_mid_left" parent="back_bottom_left_point">
+    <origin xyz="0 0 0.145" rpy="0 0 0"/>
+  </xacro:frame_point>
+  <xacro:frame_point prefix="back_mid_right" parent="back_bottom_right_point">
+    <origin xyz="0 0 0.145" rpy="0 0 0"/>
+  </xacro:frame_point>
+  <xacro:frame_point prefix="back_top_left" parent="back_mid_left_point">
+    <origin xyz="0 0 0.054" rpy="0 0 0"/>
+  </xacro:frame_point>
+  <xacro:frame_point prefix="back_top_right" parent="back_mid_right_point">
+    <origin xyz="0 0 0.054" rpy="0 0 0"/>
+  </xacro:frame_point>
+  <xacro:frame_point prefix="back_top_left_screwhole" parent="back_top_left_point">
+    <origin xyz="0.013 0.032 0" rpy="0 0 0"/>
+  </xacro:frame_point>
+  <xacro:frame_point prefix="back_top_right_screwhole" parent="back_top_right_point">
+    <origin xyz="0.013 -0.032 0" rpy="0 0 0"/>
+  </xacro:frame_point>
+  <xacro:frame_point prefix="back_top_left_screwtop" parent="back_top_left_screwhole_point">
+    <origin xyz="0 0 0.039" rpy="0 0 0"/>
+  </xacro:frame_point>
+  <xacro:frame_point prefix="back_top_right_screwtop" parent="back_top_right_screwhole_point">
+    <origin xyz="0 0 0.039" rpy="0 0 0"/>
+  </xacro:frame_point>
 </robot>
